Commit message: Fixed oscillating motion of apf and the zed2 is added to tb3_burger

File: src/dependencies/turtlebot3_description/urdf/turtlebot3_burger.gazebo.xacro (robot description, xacro)
@@ -127,23 +127,29 @@
     </sensor>
   </gazebo>
-  <gazebo reference="depth_camera">
-    <sensor name="kinect_camera" type="rgbd_camera">
+  <!-- ZED 2 as semprob.gazebo.xacro has it: one rgbd_camera with the calibrated
+       103.6 deg HFOV, 640x360 at 20 Hz and the 0.3-20 m depth range. On
+       zed_left_camera_frame because gz renders along a frame's +X, and the
+       optical frame is +Z forward. Unlike semprob, the images are stamped with
+       the optical frame: RViz's Camera display and image_geometry expect it.
+       semprob stamps the body frame for its point cloud, which gz emits in that
+       frame; this launch does not bridge /zed/points. -->
+  <gazebo reference="zed_left_camera_frame">
+    <sensor name="zed2" type="rgbd_camera">
+      <always_on>1</always_on>
+      <update_rate>20</update_rate>
+      <topic>/zed</topic>
+      <gz_frame_id>zed_left_camera_optical_frame</gz_frame_id>
       <camera>
-        <horizontal_fov>1.047</horizontal_fov>
+        <horizontal_fov>1.80799</horizontal_fov>
         <image>
           <width>640</width>
-          <height>480</height>
+          <height>360</height>
           <format>R8G8B8</format>
         </image>
         <clip>
-          <near>0.1</near>
-          <far>5.0</far>
+          <near>0.3</near>
+          <far>20.0</far>
         </clip>
       </camera>
-      <always_on>1</always_on>
-      <update_rate>30</update_rate>
-      <visualize>true</visualize>
-      <topic>camera</topic>
-      <gz_frame_id>camera_rgb_optical_frame</gz_frame_id>
     </sensor>
   </gazebo>

File: src/dependencies/turtlebot3_description/urdf/turtlebot3_burger.urdf.xacro (robot description, xacro)
@@ -150,10 +150,15 @@
     </inertial>
   </link>
-  <joint name="camera_rgb_joint" type="fixed">
-    <origin xyz="0.003 0.011 0.909" rpy="0 0 0"/>
+  <!-- ZED 2, as on the real robot (SempRob_ws semprob_robot, semprob.urdf.xacro).
+       The pose is that URDF's base_link -> zed_camera_center with the pan/tilt
+       head at zero: 1.2389 m above the ground, 5.2 deg down, 1.1 deg left. The
+       burger's base_link is 0.010 m up, so z here is 1.2289: the image is taken
+       from the real camera's viewpoint, not the burger's. -->
+  <joint name="zed_camera_center_joint" type="fixed">
+    <origin xyz="0.0426 -0.0063 1.2289" rpy="-0.0011 0.0911 0.0185"/>
     <parent link="base_link"/>
-    <child link="depth_camera"/>
+    <child link="zed_camera_center"/>
   </joint>
-  <link name="depth_camera">
+  <link name="zed_camera_center">
     <!-- Negligible mass: fixed joint, inertia contribution intentionally omitted.
            Zero inertia causes physics instability; 1e-9 is numerically safe. -->
@@ -165,13 +170,20 @@
     <visual name="visual">
       <geometry>
-        <mesh filename="file://$(find apfrl_tb3_sim)/meshes/kinect.dae" />
+        <mesh filename="file://$(find apfrl_tb3_sim)/meshes/zed2.stl"/>
       </geometry>
+      <material name="dark"/>
     </visual>
   </link>
-  <joint name="camera_rgb_optical_joint" type="fixed">
-    <origin xyz="0 0 0" rpy="-1.57 0 -1.57"/>
-    <parent link="depth_camera"/>
-    <child link="camera_rgb_optical_frame"/>
+  <joint name="zed_left_camera_joint" type="fixed">
+    <origin xyz="0 0.06 0" rpy="0 0 0"/>
+    <parent link="zed_camera_center"/>
+    <child link="zed_left_camera_frame"/>
   </joint>
-  <link name="camera_rgb_optical_frame"/>
+  <link name="zed_left_camera_frame"/>
+  <joint name="zed_left_camera_optical_joint" type="fixed">
+    <origin xyz="0 0 0" rpy="-1.5707963267948966 0 -1.5707963267948966"/>
+    <parent link="zed_left_camera_frame"/>
+    <child link="zed_left_camera_optical_frame"/>
+  </joint>
+  <link name="zed_left_camera_optical_frame"/>
 </robot>
